Commit message: updated robot urdf

File: catkin_ws/src/myrobot_description/urdf/test_robot.urdf.xacro (robot description, xacro)
@@ -31,5 +31,5 @@
     <origin xyz="0 0 0.055" rpy="0 0 0" />
     <axis xyz="0 0 1" />
-    <limit lower="0" upper="3.14" velocity="100" effort="100"/>
+    <limit lower="-1.57" upper="1.57" velocity="100" effort="100"/>
   </joint>
   <link name="body_link">
@@ -79,5 +79,5 @@
     <origin xyz="0 0 0.025" rpy="0 0 0" />
     <axis xyz="0 0 1" />
-    <limit lower="0" upper="3.14" velocity="100" effort="100"/>
+    <limit lower="-1.57" upper="1.57" velocity="100" effort="100"/>
   </joint>
   <link name="neck_link">
@@ -102,14 +102,14 @@
     <parent link="neck_link"/>
     <child link="cam_link"/>
-    <origin xyz="0 0 0.065" rpy="1.57 0 0" />
-    <axis xyz="0 0 1" />
-    <limit lower="0" upper="3.14" velocity="100" effort="100"/>
+    <origin xyz="0 0 0.065" rpy="-1.57 0 0" />
+    <axis xyz="0 0 1" />
+    <limit lower="-0.785" upper="1.57" velocity="100" effort="100"/>
   </joint>
   <!-- Here z => y and y => -z -->
   <link name="cam_link">
     <visual>
-      <origin xyz="0 0.0325 0" rpy="0 0 0"/>
-      <geometry>
-        <box size="0.05 0.065 0.08"/>
+      <origin xyz="0 -0.0325 0" rpy="0 0 0"/>
+      <geometry>
+        <box size="0.05 -0.065 0.08"/>
       </geometry>
       <material name="white" />
@@ -130,5 +130,5 @@
     <origin xyz="0.034 -0.108 0.045" rpy="1.57 0 0" />
     <axis xyz="0 0 1" />
-    <limit lower="0" upper="3.14" velocity="100" effort="100"/>
+    <limit lower="-0.26" upper="1.57" velocity="100" effort="100"/>
   </joint>
   <link name="arm_link">
@@ -157,5 +157,5 @@
     <origin xyz="0.015 -0.088 -0.005" rpy="0 0 0" />
     <axis xyz="0 0 1" />
-    <limit lower="0" upper="3.14" velocity="100" effort="100"/>
+    <limit lower="-1.57" upper="1.57" velocity="100" effort="100"/>
   </joint>
   <link name="forearm_link">

Commit message: further updated urdf with PI macro

File: catkin_ws/src/myrobot_description/urdf/test_robot.urdf.xacro (robot description, xacro)
@@ -1,4 +1,6 @@
 <?xml version="1.0"?>
 <robot xmlns:xacro="http://www.ros.org/wiki/xacro" name="hubert_robot">
+  <!-- Define Pi -->
+  <xacro:property name="PI" value="3.141592653589793" />
   <xacro:include filename="test_include.xacro" />
   <link name="world" />
@@ -31,5 +33,5 @@
     <origin xyz="0 0 0.055" rpy="0 0 0" />
     <axis xyz="0 0 1" />
-    <limit lower="-1.57" upper="1.57" velocity="100" effort="100"/>
+    <limit lower="-${PI/2}" upper="${PI/2}" velocity="100" effort="100"/>
   </joint>
   <link name="body_link">
@@ -79,5 +81,5 @@
     <origin xyz="0 0 0.025" rpy="0 0 0" />
     <axis xyz="0 0 1" />
-    <limit lower="-1.57" upper="1.57" velocity="100" effort="100"/>
+    <limit lower="-${PI/2}" upper="${PI/2}" velocity="100" effort="100"/>
   </joint>
   <link name="neck_link">
@@ -104,5 +106,5 @@
     <origin xyz="0 0 0.065" rpy="-1.57 0 0" />
     <axis xyz="0 0 1" />
-    <limit lower="-0.785" upper="1.57" velocity="100" effort="100"/>
+    <limit lower="-${PI/4}" upper="${PI/2}" velocity="100" effort="100"/>
   </joint>
   <!-- Here z => y and y => -z -->
@@ -130,5 +132,5 @@
     <origin xyz="0.034 -0.108 0.045" rpy="1.57 0 0" />
     <axis xyz="0 0 1" />
-    <limit lower="-0.26" upper="1.57" velocity="100" effort="100"/>
+    <limit lower="-${PI/6}" upper="${PI/2}" velocity="100" effort="100"/>
   </joint>
   <link name="arm_link">
@@ -157,5 +159,5 @@
     <origin xyz="0.015 -0.088 -0.005" rpy="0 0 0" />
     <axis xyz="0 0 1" />
-    <limit lower="-1.57" upper="1.57" velocity="100" effort="100"/>
+    <limit lower="-${PI/2}" upper="${PI/2}" velocity="100" effort="100"/>
   </joint>
   <link name="forearm_link">
