Commit message: Updated URDF

File: src/hubert_kinematics/urdf/test_robot.urdf.xacro (robot description, xacro)
@@ -6,5 +6,5 @@
   <link name="world" />
   <joint name="world_joint" type="fixed">
-    <origin xyz="1.5 1.0 0" rpy="0 0 0"/>
+    <origin xyz="0 0 0" rpy="0 0 0"/>
     <parent link="world"/>
     <child link="base_link"/>
@@ -92,11 +92,11 @@
     </visual>
     <collision>
-      <origin xyz="0 0 0.325" rpy="0 0 0"/>
-      <geometry>
-        <box size="0.05 0.05 0.65" />
-      </geometry>
-    </collision>
-    <xacro:inertial_box mass="0.5" x="0.05" y="0.05" z="0.65">
-      <origin xyz="0 0 0.325" rpy="0 0 0"/>
+      <origin xyz="0 0 0.0325" rpy="0 0 0"/>
+      <geometry>
+        <box size="0.05 0.05 0.065"/>
+      </geometry>
+    </collision>
+    <xacro:inertial_box mass="0.5" x="0.05" y="0.05" z="0.065">
+      <origin xyz="0 0 0.0325" rpy="0 0 0"/>
     </xacro:inertial_box>
   </link>
@@ -118,11 +118,11 @@
     </visual>
     <collision>
-      <origin xyz="0 0 0.325" rpy="0 0 0"/>
-      <geometry>
-        <box size="0.05 0.08 0.65" />
-      </geometry>
-    </collision>
-    <xacro:inertial_box mass="0.5" x="0.05" y="0.08" z="0.65">
-      <origin xyz="0 0 0.325" rpy="0 0 0"/>
+      <origin xyz="0 -0.0325 0" rpy="0 0 0"/>
+      <geometry>
+        <box size="0.05 -0.065 0.08" />
+      </geometry>
+    </collision>
+    <xacro:inertial_box mass="0.5" x="0.05" y="-0.065" z="0.08">
+      <origin xyz="0 -0.0325 0" rpy="0 0 0"/>
     </xacro:inertial_box>
   </link>
@@ -143,11 +143,11 @@
     </visual>
     <collision>
-      <origin xyz="0 0 -0.044" rpy="0 0 0"/>
-      <geometry>
-        <box size="0.025 0.025 0.088" />
-      </geometry>
-    </collision>
-    <xacro:inertial_box mass="0.5" x="0.025" y="0.025" z="0.088">
-      <origin xyz="0 0 -0.044" rpy="0 0 0"/>
+      <origin xyz="0 -0.044 0" rpy="0 0 0"/>
+      <geometry>
+        <box size="0.025 0.088 0.025"/>
+      </geometry>
+    </collision>
+    <xacro:inertial_box mass="0.5" x="0.025" y="0.088" z="0.025">
+      <origin xyz="0 -0.044 0" rpy="0 0 0"/>
     </xacro:inertial_box>
   </link>
@@ -182,9 +182,9 @@
   <joint name="end_joint" type="fixed">
     <parent link="forearm_link"/>
-    <child link="end_link"/>
+    <child link="end_effector"/>
     <origin xyz="0 -0.15 0" rpy="0 0 0" />
     <axis xyz="0 0 0" />
   </joint>
-  <link name="end_link">
+  <link name="end_effector">
     <visual>
       <origin xyz="0 -0.0125 0" rpy="0 0 0"/>
@@ -195,11 +195,11 @@
     </visual>
     <collision>
-      <origin xyz="0 0 -0.0125" rpy="0 0 0"/>
-      <geometry>
-        <box size="0.025 0.05 0.025" />
-      </geometry>
-    </collision>
-    <xacro:inertial_box mass="0.5" x="0.025" y="0.05" z="0.025">
-      <origin xyz="0 0 -0.0125" rpy="0 0 0"/>
+      <origin xyz="0 -0.0125 0" rpy="0 0 0"/>
+      <geometry>
+        <box size="0.025 0.025 0.05"/>
+      </geometry>
+    </collision>
+    <xacro:inertial_box mass="0.5" x="0.025" y="0.025" z="0.05">
+      <origin xyz="0 -0.0125 0" rpy="0 0 0"/>
     </xacro:inertial_box>
   </link>

Commit message: More changes to urdf file

File: src/hubert_kinematics/urdf/test_robot.urdf.xacro (robot description, xacro)
@@ -120,8 +120,8 @@
       <origin xyz="0 -0.0325 0" rpy="0 0 0"/>
       <geometry>
-        <box size="0.05 -0.065 0.08" />
-      </geometry>
-    </collision>
-    <xacro:inertial_box mass="0.5" x="0.05" y="-0.065" z="0.08">
+        <box size="0.05 0.065 0.08" />
+      </geometry>
+    </collision>
+    <xacro:inertial_box mass="0.5" x="0.05" y="0.065" z="0.08">
       <origin xyz="0 -0.0325 0" rpy="0 0 0"/>
     </xacro:inertial_box>

Commit message: finalizing 3d projection

File: src/hubert_kinematics/urdf/test_robot.urdf.xacro (robot description, xacro)
@@ -141,4 +141,15 @@
         </inertial>
     </link>
+    <joint name="camera_joint" type="fixed">
+        <parent link="cam_link" />
+        <child link="camera_link" />
+        <origin rpy="0 1.5707963267948966 0" xyz="0 0 0" />
+    </joint>
+    <link name="camera_link">
+        <inertial>
+            <mass value="0" />
+            <inertia ixx="0" ixy="0" ixz="0" iyy="0" iyz="0" izz="0" />
+        </inertial>
+    </link>
     <joint name="shoulder_joint" type="revolute">
         <parent link="shoulder_link" />

Commit message: 3d projection done

File: src/hubert_kinematics/urdf/test_robot.urdf.xacro (robot description, xacro)
@@ -144,5 +144,5 @@
         <parent link="cam_link" />
         <child link="camera_link" />
-        <origin rpy="0 1.5707963267948966 0" xyz="0 0 0" />
+        <origin rpy="0 1.5707963267948966 0" xyz="0 -0.07 0" />
     </joint>
     <link name="camera_link">
